File: ShiftDriverMotherboard64.sch (KiCad schematic (older format))
At the start: 21 parts, among them J1 PWR_SCREWTERM, Q1 Q_NPN_EBC, SW1 5V_SW, SW2 PWR_SW, U1 ShiftDriver, U10 LM7805_TO220, U11 CD74HC243, U2 ShiftDriver, U3 ShiftDriver, U4 ShiftDriver, U5 ShiftDriver, U6 ShiftDriver, U7 ShiftDriver, U8 ShiftDriver, U9 TEENSY_3.6_MINIMAL

Commit message: finished scheamtic
Parts:
- removed SW2: PWR_SW, symbol Switch:SW_SPST
- added C1, C9: 10uf, Capacitor_THT:CP_Radial_D5.0mm_P2.00mm, symbol Device:CP
- added C2, C7, C8: 0.1uf, Capacitor_THT:C_Disc_D3.0mm_W2.0mm_P2.50mm, symbol Device:C
- added C3, C4, C5, C6: 470uf, Capacitor_THT:CP_Radial_D10.0mm_P5.00mm, symbol Device:CP
- added D4: CLR_LED, LED_THT:LED_D5.0mm, symbol Device:LED
- added D5: EN_LED, LED_THT:LED_D5.0mm, symbol Device:LED
- added D6: 1N4001, Diode_THT:D_DO-41_SOD81_P7.62mm_Horizontal, symbol Device:D
- added D7: LOCK_IND, LED_THT:LED_D5.0mm, symbol Device:LED
- added D8: BOOT_IND, LED_THT:LED_D5.0mm, symbol Device:LED_Dual_2pin
- added J2: PWR OPTION HEADER, Connector_PinHeader_2.54mm:PinHeader_2x04_P2.54mm_Vertical, symbol Connector_Generic:Conn_02x04_Odd_Even
- added J3: VTEENSY, HammerheadAudio:Phoenix_Stacked, symbol Connector:Conn_01x02_Female
- added Q2: Q_NPN_EBC, Package_TO_SOT_THT:TO-92L_Inline_Wide, symbol Device:Q_NPN_EBC
- added R4, R6, R7: 1k, HammerheadAudio:R_THT_P7.62, symbol Device:R
- added R5: 10k, HammerheadAudio:R_THT_P7.62, symbol Device:R
- added SW2: BOOT_MODE, HammerheadAudio:Tayda_Slide_SPDT, symbol Switch:SW_SPDT
- added SW3: MUTE_SW, HammerheadAudio:Tayda_Slide_SPDT, symbol Switch:SW_SPDT
- added U12: EAPLRAA4, HammerheadAudio:EAPLRAA4, symbol Interface_Optical:TSDP341xx
- D2: value 5V_IND -> TEENSY_PWR_IND
- J1: footprint (none) -> HammerheadAudio:ScrewTerm+Phoenix_30A_7.62mm_1x2
- SW1: value 5V_SW -> TEENSY_PWR; footprint (none) -> HammerheadAudio:Tayda_Slide_SPDT
Connections:
- net +5V: now also C1.1, C2.1, Q2.3 (C); no longer U10.3 (VO)
- net CLK_PIN: now also U9.35 (13_SCK0_LED)
- net CLR: now also R4.1
- net CLR_PIN: now also U9.11 (9_PWM_RX2_CS0)
- net CS_PIN: now also U9.12 (10_PWM_TX2_CS0)
- net DAT_PIN: now also U9.13 (11_MOSI0)
- net EN: now also Q2.1 (E); no longer Q1.3 (C), R1.2
- net EN_PIN: now also U9.10 (8_TX3_miso0_sda0), R5.2; no longer Q1.2 (B)
- net GND: now also J1.1 (Pin_1), C1.2, C2.2, C3.2, C4.2, C5.2, C6.2, C7.2, C8.2, C9.2, D4.1 (K), D5.1 (K), D7.1 (K), J3.1 (Pin_1), SW2.3 (C), SW3.3 (C), U12.2 (GND); no longer D1.2 (A), J1.2 (Pin_2), Q1.1 (E)
- net VDD: now also J1.2 (Pin_2), C3.1, C4.1, C5.1, C6.1, C7.1, C8.1, J2.1 (Pin_1), J2.3 (Pin_3); no longer D1.1 (K), SW1.2 (B)
- net +3V3: now reaches U9.15 (3.3V)
- net +3V3: now also U9.46 (3.3V_max250mA), U12.3 (Vs)
- net SPDIF: now reaches U9.37 (15_A1_CS0_Touch)
- net SPDIF: now also U12.1 (OUT)
- net at U9.43 (21_A7_PWM_CS0_sck1): now also SW3.2 (B)
- net at U9.44 (22_A8_PWM_Touch): now also SW2.2 (B)
- net BOOT_IND2: now reaches U9.7 (5_PWM_tx1_miso1)
- net BOOT_IND2: now also R7.2
- net BOOT_IND1: now reaches U9.8 (6_PWM)
- net BOOT_IND1: now also D8.2 (AK)
- net LOCK_PIN: now reaches U9.9 (7_RX3_miso0_scl0)
- net LOCK_PIN: now also R6.1
- net at SW1.3 (C): no longer U10.1 (VI)
- new net: J2.5 (Pin_5), J2.7 (Pin_7), J3.2 (Pin_2)
- new net: Q1.3 (C), Q2.2 (B), R1.2
- new net: D1.1 (K), SW1.2 (B), U10.3 (VO)
- new net: C9.1, D6.1 (K), U10.1 (VI)
- new net: D5.2 (A), Q1.1 (E)
- new net: Q1.2 (B), R5.1
- new net: D4.2 (A), R4.2
- new net: D8.1 (KA), R7.1
- new net: D7.2 (A), R6.2
- new net VSPK_TO_5V: D1.2 (A), J2.4 (Pin_4), J2.8 (Pin_8)
- new net VSPK_TO_REG: D6.2 (A), J2.2 (Pin_2), J2.6 (Pin_6)
- no-connect marks 1 -> 36
Other:
- moved on the sheet: D2, D3, J1, Q1, R1, R2, R3, U10, U11, U9
