File: ShiftDriverMotherboard64.sch (KiCad schematic (older format))
At the start: 47 parts, among them J1 - V_SPK_IN +, J2 PWR OPTION HEADER, J3 V_TNSY_IN, Q1 Q_NPN_EBC, Q2 Q_NPN_EBC, SW1 TEENSY_PWR, SW2 BOOT_MODE, SW3 MUTE_SW, U1 ShiftDriver, U10 LM7805_TO220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

Commit message: finished layout tweaks, made gerbers
Parts:
- gave numbers to parts that had none: 1
Changed lines of the file:
@@
 Connection ~ 8100 4700
 $Comp
-L Device:C C?
+L Device:C C10
 U 1 1 5EF13F83
 P 2000 3900
-F 0 "C?" H 2115 3946 50  0000 L CNN
+F 0 "C10" H 2115 3946 50  0000 L CNN
 F 1 "0.1uf" H 2115 3855 50  0000 L CNN
 F 2 "Capacitor_THT:C_Disc_D3.0mm_W2.0mm_P2.50mm" H 2038 3750 50  0001 C CNN

Commit message: ready for printing
Parts:
- J1: value - V_SPK_IN + -> - VSPK_IN +
Connections:
- net +3V3: no longer U9.15 (3.3V)
- no-connect marks 36 -> 37
Other:
- moved on the sheet: C1, C10, C2, C8, C9, D1, D2, D3, D6, D9, J1, J2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
