File: ShiftDriverMotherboard64.kicad_pcb (KiCad board)
At the start: 2 copper layers, 230 x 180 mm, 55 parts, among them J1 - VSPK_IN +, J2 PWR OPTION HEADER, J3 V_TNSY_IN, Q1 Q_NPN_EBC, Q2 Q_NPN_EBC, SW1 TEENSY_PWR, SW2 BOOT_MODE, SW3 MUTE_SW, U1 ShiftDriver, U10 LM7805_TO220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

Commit message: finished first draft of layout
Parts:
- added C10: 0.1uf, Capacitor_THT:C_Disc_D3.0mm_W2.0mm_P2.50mm, F.Cu at (34.2, 182.8)
- J1: value - VSPK_IN + -> - V_SPK_IN +
Connections:
- D8 pad 2: BOOT_IND1 -> BOOT_IND2
- R7 pad 2: BOOT_IND2 -> BOOT_IND1
Routing:
- net +5V: track 0.00 -> 1080.9 mm
- net CS: track 0.00 -> 568.8 mm
- net CLR: track 0.00 -> 453.8 mm
- net EN: track 0.00 -> 442.0 mm
- net S_CLK: track 0.00 -> 419.9 mm
- net D5: track 0.00 -> 221.6 mm
- net Net-(SW3-Pad2): track 0.00 -> 156.3 mm
- net Net-(SW2-Pad2): track 0.00 -> 132.5 mm
- net D1: track 0.00 -> 91.0 mm
- net D8: track 0.00 -> 74.6 mm
- net D4: track 0.00 -> 73.5 mm
- net D6: track 0.00 -> 61.7 mm
- net D7: track 0.00 -> 60.5 mm
- net D2: track 0.00 -> 60.3 mm
- net D3: track 0.00 -> 59.9 mm
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
Commit message: finished layout tweaks, made gerbers
Parts:
- added HH_LOGO_32x16: , HammerheadAudio:HH_LOGO_32x16, B.Cu at (219.5, 21.8)
- J1: value - V_SPK_IN + -> - VSPK_IN +
Routing:
- net +5V: track 1080.9 -> 1079.9 mm
Other:
- board text added: "! YOUR SILENCE IS DIRESPECTFUL !"
- board text added: "- VSPK_IN +"
- board text added: "64 X 1-BIT AUDIO CHANNEL DRIVER"
- board text added: "HAMMERHEAD AUDIO - SHIFT DRIVER MOTHERBOARD 64 V0.1 - EMMETT PALAIMA - 2020"
- board text added: "MUTE<—>UNMUTE"
- board text removed: "MUTE<——>UNMUTE"

Commit message: ready for printing
Parts:
- moved C9 3.61 mm to (157.2, 152.0)
- moved D1 3.61 mm to (165.2, 152.0)
- moved D6 3.61 mm to (161.5, 152.0)
- moved C6 2.00 mm to (195.3, 157.8)
- moved C7 2.00 mm to (195.3, 153.2)
- moved U10 2.00 mm to (172.2, 153.0)
- moved J2 0.50 mm to (173.5, 166.0)
Connections:
- U9 pad 15: +3V3 -> Net-(U9-Pad15)
Routing:
- net +5V: track 1079.9 -> 1203.3 mm
- net +3V3: track 53.7 -> 32.1 mm
- net D3: track 59.9 -> 70.4 mm
- net D7: track 60.5 -> 69.1 mm
- net D2: track 60.3 -> 67.3 mm
- net D6: track 61.7 -> 68.5 mm
- net VSPK_TO_REG: track 22.4 -> 27.6 mm
- net VSPK_TO_5V: track 22.1 -> 25.0 mm
- net D8: track 74.6 -> 72.0 mm
- net S_CLK: track 419.9 -> 421.4 mm
- net VDD: track 40.8 -> 39.6 mm
- net Net-(D1-Pad1): track 41.0 -> 39.9 mm
- net Net-(C9-Pad1): track 18.0 -> 18.8 mm
- net CS: track 568.8 -> 568.3 mm

Commit message: fixed shift driver footprint and resized board
Parts:
- removed the H3 at (15.0, 185.0)
- removed the H3 at (235.0, 100.0)
- removed the H3 at (235.0, 185.0)
- removed the H3 at (15.0, 100.0)
- removed the H3 at (125.0, 15.0)
- removed the H3 at (125.0, 185.0)
- removed the H3 at (235.0, 15.0)
- removed HH_LOGO_13.5x6.75: , HammerheadAudio:HH_LOGO_13.5x6.75
- removed the HH_LOGO_32x16 at (219.5, 21.8)
- added H3: M3/#4-40, HammerheadAudio:M3_MOUNT, F.Cu at (15.0, 195.0)
- added H3: M3/#4-40, HammerheadAudio:M3_MOUNT, F.Cu at (255.0, 105.0)
- added H3: M3/#4-40, HammerheadAudio:M3_MOUNT, F.Cu at (255.0, 195.0)
- added H3: M3/#4-40, HammerheadAudio:M3_MOUNT, F.Cu at (15.0, 105.0)
- added H3: M3/#4-40, HammerheadAudio:M3_MOUNT, F.Cu at (135.0, 15.0)
- added H3: M3/#4-40, HammerheadAudio:M3_MOUNT, F.Cu at (135.0, 195.0)
- added H3: M3/#4-40, HammerheadAudio:M3_MOUNT, F.Cu at (255.0, 15.0)
- added HH_LOGO_32x16: , HammerheadAudio:HH_LOGO_32x16, F.Cu at (74.0, 169.8)
- added HH_LOGO_32x16: , HammerheadAudio:HH_LOGO_32x16, B.Cu at (237.5, 21.8)
- moved C6 22.8 mm to (215.8, 167.8)
- moved C7 22.8 mm to (215.8, 163.2)
- moved C1 22.4 mm to (160.0, 192.5)
- moved C3 22.4 mm to (240.8, 191.0)
- moved C4 22.4 mm to (240.8, 178.0)
- moved C5 22.4 mm to (240.8, 165.0)
- moved D2 22.4 mm to (168.2, 192.0)
- moved D3 22.4 mm to (205.5, 192.0)
- moved D9 22.4 mm to (193.5, 192.0)
- moved J1 22.4 mm to (219.8, 173.0)
- moved J3 22.4 mm to (179.0, 192.0)
- moved R2 22.4 mm to (164.5, 188.5)
- moved R3 22.4 mm to (209.2, 188.5)
- moved R8 22.4 mm to (189.8, 188.5)
- moved J2 21.4 mm to (193.5, 173.8)
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Routing:
- net +5V: track 1203.3 -> 0.00 mm
- net CS: track 568.3 -> 0.00 mm
- net CLR: track 453.8 -> 0.00 mm
- net EN: track 442.2 -> 0.00 mm
- net S_CLK: track 421.4 -> 0.00 mm
- net D5: track 221.6 -> 0.00 mm
- net Net-(SW3-Pad2): track 156.3 -> 0.00 mm
- net Net-(SW2-Pad2): track 132.5 -> 0.00 mm
- net D1: track 90.6 -> 0.00 mm
- net D4: track 73.5 -> 0.00 mm
- net D8: track 72.0 -> 0.00 mm
- net D3: track 70.4 -> 0.00 mm
- net D7: track 69.1 -> 0.00 mm
- net D6: track 68.5 -> 0.00 mm
- net D2: track 67.3 -> 0.00 mm
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Other:
- board size 230 x 180 mm -> 250 x 190 mm

Commit message: finished new layout
Parts:
- added HH_LOGO_32x16: , HammerheadAudio:HH_LOGO_32x16, F.Cu at (78.0, 169.8)
- moved HH_LOGO_32x16 4.00 mm to (78.0, 169.8)
Routing:
- net +5V: track 0.00 -> 1334.2 mm
- net CS: track 0.00 -> 627.3 mm
- net CLR: track 0.00 -> 503.4 mm
- net EN: track 0.00 -> 472.3 mm
- net S_CLK: track 0.00 -> 464.5 mm
- net D5: track 0.00 -> 227.5 mm
- net Net-(SW3-Pad2): track 0.00 -> 169.7 mm
- net Net-(SW2-Pad2): track 0.00 -> 146.7 mm
- net D1: track 0.00 -> 110.3 mm
- net D8: track 0.00 -> 82.1 mm
- net D4: track 0.00 -> 81.0 mm
- net D7: track 0.00 -> 75.3 mm
- net D6: track 0.00 -> 74.0 mm
- net D2: track 0.00 -> 66.9 mm
- net D3: track 0.00 -> 65.7 mm
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Other:
- outline, holes or cut-outs redrawn
- board text added: "HAMMERHEAD AUDIO - SHIFT DRIVER MOTHERBOARD 64 V0.2 - EMMETT PALAIMA - 2020"
- board text removed: "HAMMERHEAD AUDIO - SHIFT DRIVER MOTHERBOARD 64 V0.1 - EMMETT PALAIMA - 2020"

Commit message: final tweaks, made gerbers
Routing:
- net +5V: track 1334.2 -> 1324.4 mm
Changed lines of the file:
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@@
     (39 F.Mask user)
     (40 Dwgs.User user)
-    (41 Cmts.User user hide)
+    (41 Cmts.User user)
     (42 Eco1.User user)
     (43 Eco2.User user)
@@
   )
   (setup
-    (last_trace_width 0.25)
+    (last_trace_width 1)
     (user_trace_width 0.5)
     (user_trace_width 1)
@@
   (segment (start 71.8 62.2) (end 200.8 62.2) (width 1) (layer F.Cu) (net 33))
   (segment (start 200.8 62.2) (end 205.8 67.2) (width 1) (layer F.Cu) (net 33))
-  (segment (start 205.8 67.2) (end 205.8 92) (width 1) (layer F.Cu) (net 33))
-  (segment (start 199.64 98.16) (end 196.54 98.16) (width 1) (layer F.Cu) (net 33))
-  (segment (start 205.8 92) (end 199.64 98.16) (width 1) (layer F.Cu) (net 33))
+  (segment (start 138.54 30.16) (end 158.84 30.16) (width 1) (layer F.Cu) (net 33))
+  (segment (start 170.2 18.8) (end 193 18.8) (width 1) (layer F.Cu) (net 33))
+  (segment (start 158.84 30.16) (end 170.2 18.8) (width 1) (layer F.Cu) (net 33))
+  (segment (start 200.4 87.2) (end 205.8 81.8) (width 1) (layer F.Cu) (net 33))
+  (segment (start 193.2 87.2) (end 200.4 87.2) (width 1) (layer F.Cu) (net 33))
+  (segment (start 205.8 67.2) (end 205.8 81.8) (width 1) (layer F.Cu) (net 33))
   (segment (start 49.5 130.2) (end 22.54 103.24) (width 1) (layer F.Cu) (net 33))
   (segment (start 199 130.2) (end 49.5 130.2) (width 1) (layer F.Cu) (net 33))
   (segment (start 205.6 136.8) (end 199 130.2) (width 1) (layer F.Cu) (net 33))
   (segment (start 205.6 152) (end 205.6 136.8) (width 1) (layer F.Cu) (net 33))
-  (segment (start 201.600011 155.999989) (end 205.6 152) (width 1) (layer F.Cu) (net 33))
-  (segment (start 145.200011 155.999989) (end 201.600011 155.999989) (width 1) (layer F.Cu) (net 33))
-  (segment (start 138.4 162.8) (end 145.200011 155.999989) (width 1) (layer F.Cu) (net 33))
-  (segment (start 138.54 30.16) (end 158.84 30.16) (width 1) (layer F.Cu) (net 33))
-  (segment (start 170.2 18.8) (end 193 18.8) (width 1) (layer F.Cu) (net 33))
-  (segment (start 158.84 30.16) (end 170.2 18.8) (width 1) (layer F.Cu) (net 33))
+  (segment (start 142.8 167.2) (end 154.25 155.75) (width 1) (layer F.Cu) (net 33))
+  (segment (start 201.85 155.75) (end 205.6 152) (width 1) (layer F.Cu) (net 33))
+  (segment (start 154.25 155.75) (end 201.85 155.75) (width 1) (layer F.Cu) (net 33))
   (segment (start 209.25 188.5) (end 226.5 188.5) (width 1) (layer F.Cu) (net 35))
   (segment (start 227.42 189.42) (end 227.42 192.25) (width 1) (layer F.Cu) (net 35))
@@
     (polygon
       (pts
-        (xy 232.5 195) (xy 243 195) (xy 243 106) (xy 249 106) (xy 249 88)
-        (xy 244 88) (xy 244 38) (xy 249 38) (xy 249 20) (xy 243 20)
-        (xy 223.5 20) (xy 223.5 38) (xy 192 38) (xy 192 20) (xy 186 20)
-        (xy 186 38) (xy 134 38) (xy 134 20) (xy 128 20) (xy 128 38)
-        (xy 76 38) (xy 76 20) (xy 70 20) (xy 70 48) (xy 217 48)
-        (xy 217 106) (xy 192 106) (xy 192 88) (xy 186 88) (xy 186 106)
-        (xy 134 106) (xy 134 88) (xy 128 88) (xy 128 106) (xy 76 106)
-        (xy 76 88) (xy 70 88) (xy 70 116) (xy 217 116) (xy 217 170)
+        (xy 232.5 195) (xy 243 195) (xy 243 178) (xy 243 161) (xy 244 161)
+        (xy 244 106) (xy 249 106) (xy 249 88) (xy 244 88) (xy 244 38)
+        (xy 249 38) (xy 249 20) (xy 243 20) (xy 223.5 20) (xy 223.5 38)
+        (xy 192 38) (xy 192 20) (xy 186 20) (xy 186 38) (xy 134 38)
+        (xy 134 20) (xy 128 20) (xy 128 38) (xy 76 38) (xy 76 20)
+        (xy 70 20) (xy 70 50) (xy 210 50) (xy 210 106) (xy 192 106)
+        (xy 192 88) (xy 186 88) (xy 186 106) (xy 134 106) (xy 134 88)
+        (xy 128 88) (xy 128 106) (xy 76 106) (xy 76 88) (xy 70 88)
+        (xy 70 118) (xy 210 118) (xy 210 153) (xy 217 153) (xy 217 170)
         (xy 224 170) (xy 224 171.25) (xy 232.5 171.25)
       )
@@
     (polygon
       (pts
-        (xy 260 200) (xy 221 200) (xy 221 196) (xy 244 196) (xy 244 107)
-        (xy 250 107) (xy 250 87) (xy 245 87) (xy 245 39) (xy 250 39)
-        (xy 250 19) (xy 222 19) (xy 222 37) (xy 193 37) (xy 193 19)
-        (xy 185 19) (xy 185 37) (xy 135 37) (xy 135 19) (xy 127 19)
-        (xy 127 37) (xy 77 37) (xy 77 19) (xy 69 19) (xy 69 49)
-        (xy 216 49) (xy 216 105) (xy 193 105) (xy 193 87) (xy 185 87)
-        (xy 185 105) (xy 135 105) (xy 135 87) (xy 127 87) (xy 127 105)
-        (xy 77 105) (xy 77 87) (xy 69 87) (xy 69 117) (xy 216 117)
-        (xy 216 171) (xy 217 171) (xy 217 200) (xy 86 200) (xy 10 200)
-        (xy 10 10) (xy 249 10) (xy 260 10) (xy 260 49.25) (xy 260 94.5)
+        (xy 260 200) (xy 221 200) (xy 221 196) (xy 244 196) (xy 244 162)
+        (xy 245 162) (xy 245 107) (xy 250 107) (xy 250 87) (xy 245 87)
+        (xy 245 39) (xy 250 39) (xy 250 19) (xy 222 19) (xy 222 37)
+        (xy 193 37) (xy 193 19) (xy 185 19) (xy 185 37) (xy 135 37)
+        (xy 135 19) (xy 127 19) (xy 127 37) (xy 77 37) (xy 77 19)
+        (xy 69 19) (xy 69 51) (xy 209 51) (xy 209 105) (xy 193 105)
+        (xy 193 87) (xy 185 87) (xy 185 105) (xy 135 105) (xy 135 87)
+        (xy 127 87) (xy 127 105) (xy 77 105) (xy 77 87) (xy 69 87)
+        (xy 69 119) (xy 209 119) (xy 209 154) (xy 216 154) (xy 216 171)
+        (xy 217 171) (xy 217 200) (xy 86 200) (xy 10 200) (xy 10 10)
+        (xy 249 10) (xy 260 10) (xy 260 49.25) (xy 260 94.5)
       )
     )
